Commit message: Implemented simulation startup and shutdown scripts for convenience. Made modifications to some simulation launch files, as well as default configs for rviz again for convenience.

File: src/urdf_description/urdf/URDF.xacro (robot description, xacro)
@@ -632,5 +632,5 @@
   <parent link="hull_top_1"/>
   <child link="lidar_link"/>
-  <origin xyz="-0.2999999663283473 0 0.25" rpy="0 0 0"/>
+  <origin xyz="-0.2999999663283473 0 0.10" rpy="0 0 0"/>
 </joint>
 </robot>

Commit message: Initial overhaul with Codex

File: src/urdf_description/urdf/URDF.xacro (robot description, xacro)
@@ -506,4 +506,17 @@
   </collision>
 </link>
+<!-- Update these zero-offset joints after measuring the installed sensors. -->
+<link name="imu_link"/>
+<joint name="imu_joint" type="fixed">
+  <parent link="base_link"/>
+  <child link="imu_link"/>
+  <origin xyz="0 0 0" rpy="0 0 0"/>
+</joint>
+<link name="gps_link"/>
+<joint name="gps_joint" type="fixed">
+  <parent link="base_link"/>
+  <child link="gps_link"/>
+  <origin xyz="0 0 0" rpy="0 0 0"/>
+</joint>
 <joint name="left_pushbar_joint" type="fixed">
   <origin xyz="-0.18877 0.09187 -0.1479" rpy="0 0 0"/>
