Commit message: Hardware-free follow simulation, follow smoke test, Jetson fixes
- fake_robot integrates /cmd_vel_mux into a unicycle pose around a GPS
  datum and publishes /odom_rf2o, /imu/data (magnetic yaw), robot GPS,
  an empty scan and ground truth on /sim/pose. fake_beacon walks a
  waypoint path on /gps/beacon/fix. bringup.launch.py sim:=true runs
  them with the real robot model, EKFs, navsat and Nav2.
- follow_smoke_test.py plays the beacon and checks four phases:
  approach and stop near 3 m, follow a 12 m walk, halt after beacon
  fixes stop, resume when they return. Passes 3 of 3 runs.
- Scans are stamped 0.1 s back, as rplidar_ros does. Scans stamped
  ahead of TF made the costmap's MessageFilter wait asynchronously,
  and on tf2_ros 0.25.23 that deadlocked controller_server's TF
  listener (gdb: MessageFilter::add -> addTransformableRequest vs
  setTransform -> testTransformableRequests), freezing the robot.
- Nav2 controller: Regulated Pure Pursuit instead of MPPI at 10 Hz;
  EKFs at 30 Hz and navsat at 10 Hz to fit the Orin Nano CPU; path
  transform_tolerance 0.5 s.
- follow_manager: rename self.handle (clashes with rclpy Node.handle).
- URDF: add a gps link (zero offset until the antenna is measured).

Co-Authored-By: Claude Opus 5.5 <noreply@anthropic.com>

File: src/urdf_description/urdf/URDF.xacro (robot description, xacro)
@@ -484,4 +484,12 @@
   </collision>
 </link>
+<!-- GPS antenna frame used by navsat_transform_node. TODO: measure the real
+     antenna offset from base_link; zero until then. -->
+<link name="gps"/>
+<joint name="gps_joint" type="fixed">
+  <parent link="base_link"/>
+  <child link="gps"/>
+  <origin xyz="0 0 0" rpy="0 0 0"/>
+</joint>
 <link name="lidar_link">
   <inertial>

Commit message: Set the measured GPS antenna offset in the URDF
Co-Authored-By: Claude Opus 5.5 <noreply@anthropic.com>

File: src/urdf_description/urdf/URDF.xacro (robot description, xacro)
@@ -484,11 +484,14 @@
   </collision>
 </link>
-<!-- GPS antenna frame used by navsat_transform_node. TODO: measure the real
-     antenna offset from base_link; zero until then. -->
+<!-- GPS antenna frame used by navsat_transform_node. Measured on the robot
+     (2026-09-26): 16 cm forward of the wheel midpoint, on the center line,
+     63 cm above the ground. base_link sits 0.169 m above the ground (bottom
+     of the wheel meshes), so z = 0.63 - 0.169. x is forward (REP-103), which
+     is how odometry moves base_link. -->
 <link name="gps"/>
 <joint name="gps_joint" type="fixed">
   <parent link="base_link"/>
   <child link="gps"/>
-  <origin xyz="0 0 0" rpy="0 0 0"/>
+  <origin xyz="0.16 0 0.461" rpy="0 0 0"/>
 </joint>
 <link name="lidar_link">
